File: diodes.kicad_pcb (KiCad board)
At the start: 2 copper layers, 13 parts

Commit message: schematics
Parts:
- added REF**: D_MicroSMP_AK, Diode_SMD:D_MicroSMP_AK, F.Cu at (112.2, 80.7)
- REF**: value D_SMF -> D_SMF / DO-219
- moved REF** 48.2 mm to (111.7, 87.0)
