File: Sensors.kicad_sch (KiCad schematic)
At the start: 22 parts, among them U3 INA226, U6 AS333

Commit message: Current sense: INA226 -> AS333 on ADC, battery divider, port routed U6 cluster
Schematic (Sensors, uC):
- INA226 path (U3, R25, R27, C23, C24, R28, R29, C25) DNP and excluded from board.
- AS333 low-side amplifier (U6, R39-R42, C29, C32) fitted; V- and C29 return to GND.
  Rescaled R41 43k / R42 226k: ADC_I = 0.64 V + 21.5 mV/A, -29..+44 A in 0..1.6 V
  (ESP32-S3 ADC 6 dB). C26 footprint kept, DNP.
- ADC_I via R51 1k + C36 100n to GPIO5 (ADC1_CH4) and J4.11 (MCU head, spare pin).
- Battery voltage: R52 470k / R53 11k / C37 100n from BT+ to GPIO6 (ADC1_CH5) as
  ADC_Vbat (ratio 43.7: 58.4 V -> 1.34 V), replacing the INA226 VBUS reading.

PCB:
- U6 cluster placement and local copper ported from branch fets-to-tdson8, incl.
  the Kelvin lines to R26; R51/C36 at the branch's series-R/filter spot below U2.
- Removed the old cluster copper and stale BuckGND tracks shorting U6/C29/R42.
- Branch +3.3V feed and long OUT_ISENSE run not ported (main's routing diverged);
  +3.3V to U6, OUT_ISENSE to R51 and ADC_I to GPIO5/J4.11 remain to be routed.

doc/reviews/2026-09-30-schematic: per-sheet schematic review, taken before the
current-sense change.
Parts:
- added C36, C37: 100nF, 25V, Capacitor_SMD:C_0805_2012Metric, symbol Device:C_Small
- added R51: 1k, Resistor_SMD:R_0805_2012Metric, symbol Device:R_Small
- added R52: 470k, 1%, Resistor_SMD:R_0805_2012Metric, symbol Device:R_Small
- added R53: 11k, 1%, Resistor_SMD:R_0805_2012Metric, symbol Device:R_Small
- C23, C24, C25, R25, R27, R28, R29, U3: now not fitted
- C29, C32, R39, R40, U6: now fitted
- R41: value 75k -> 43k, 1%; now fitted
- R42: value 150k -> 226k, 1%; now fitted
Connections:
- net BuckGND is gone; now on net GND: C29.2, U6.2 (V-)
- net BT+: now also R52.1
- net GND: now also C36.2, C37.2, R53.2
- net at C32.1, R41.1, U6.4: now also R51.1
- new net ADC_I: C36.1, R51.2
- new net ADC_Vbat: C37.1, R52.2, R53.1
Other:
- note added: "ADC_I = 0.64 V + 21.5 mV/A (Rs 0.5 mOhm, G = 43) -29 A .. +44 A -> 0 .. 1.6 V (ESP32-S3 ADC 6 dB) 1k + 100n at the pin: GPIO5 boot glitch, ADC guideline"
- note added: "Battery voltage (replaces INA226 VBUS) ratio 43.7: 58.4 V -> 1.34 V, 70 V -> 1.60 V 80 V fault -> 1.83 V; drain 0.12 mA @ 58 V"
- note removed: "TODO: use GND here instead of BuckGND"
