File: ExtPort.kicad_sch (KiCad schematic)
At the start: 15 parts, among them J5 VE.Direct port (JST-PH 4), U7 SN74LVC1G125DBVR, U8 SN74LVC1G17DBVR

Commit message: ExtPort: power TX buffer from V+ (ISO1042 TXD <= VCC1+0.5V); plan: review 2 findings
Parts:
- C34: Desc ExtPort bypass -> ExtPort bypass (U7)
Connections:
- net +3.3V: no longer C34.1, U7.5 (VCC)
- net EXT_VP: now reaches C33.1, D19.2 (A2), D22.1 (K), J5.4 (Pin_4)
- net EXT_VP: now also C34.1, U7.5 (VCC)
Other:
- note added: "External comms port, VE.Direct pinout (plans/ext-comms-port.md) J5 pin | signal | dir (Fugu view) | notes 1 | GND | - | logic GND = Bat-; non-isolated 2 | RX | in | 3.3 V logic, 5.5 V tolerant (U8), idles high (R50) 3 | TX | out | 3.3 V push-pull via 220R, Hi-Z unless EXT_TX_OE_N low (R46 pull-up) 4 | V+ | out | EXT_VP: +3.3V via Schottky D22, always on; ~2.85 V at 170 mA on a 3.2 V rail | | | (3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"
- note removed: "External comms port, VE.Direct pinout (plans/ext-comms-port.md) J5 pin | signal | dir (Fugu view) | notes 1 | GND | - | logic GND = Bat-; non-isolated 2 | RX | in | 3.3 V logic, 5.5 V tolerant (U8), idles high (R50) 3 | TX | out | 3.3 V push-pull via 220R, Hi-Z unless EXT_TX_OE_N low (R46 pull-up) 4 | V+ | out | +3.3V via Schottky D22, always on; ~2.85 V at 170 mA (VF ~0.35 V typ) MCU: EXT_TX GPI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"

Commit message: ExtPort: drop TVS D19 on V+; C33 is the pin-4 ESD sink
Parts:
- removed D19: LESD5D5.0CT1G, Diode_SMD:D_SOD-523, symbol Device:D_TVS

Commit message: ExtPort: drop C34; C33 bypasses U7 on EXT_VP
Parts:
- removed C34: 100nF, X7R, 25V, Capacitor_SMD:C_0805_2012Metric, symbol Device:C_Small

Commit message: Remove D22: V+ direct from 3.3 V; plan: non-isolated ±70 V adapters, 60 V GND-fault requirement
Every ±60 V-class CAN/RS-485 transceiver needs >= 3.0 V; D22 left 2.7-2.95 V.
Adapter candidates from the 2026-09-30 survey (~/research/fugu2-comms-transceivers):
TCAN1042H(+boost) / MAX33053E / LTC2875 for CAN, THVD2410 with DE-from-TX for RS-485.
Parts:
- removed D22: MSS1P4-M3/89A, Diode_SMD:D_MicroSMP_LargeCathode, symbol Device:D_Schottky
Connections:
- net EXT_VP is gone; now on net +3.3V: C33.1, J5.4 (Pin_4), U7.5 (VCC)
Other:
- note added: "External comms port, VE.Direct pinout (plans/ext-comms-port.md) J5 pin | signal | dir (Fugu view) | notes 1 | GND | - | logic GND = Bat-; non-isolated 2 | RX | in | 3.3 V logic, 5.5 V tolerant (U8), idles high (R50) 3 | TX | out | 3.3 V push-pull via 220R, Hi-Z unless EXT_TX_OE_N low (R46 pull-up) 4 | V+ | out | +3.3V rail direct, always on (Fab, 2026-09-30). C33 at pin 4 = ESD sink + U7 bypass M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"
- note removed: "External comms port, VE.Direct pinout (plans/ext-comms-port.md) J5 pin | signal | dir (Fugu view) | notes 1 | GND | - | logic GND = Bat-; non-isolated 2 | RX | in | 3.3 V logic, 5.5 V tolerant (U8), idles high (R50) 3 | TX | out | 3.3 V push-pull via 220R, Hi-Z unless EXT_TX_OE_N low (R46 pull-up) 4 | V+ | out | EXT_VP: +3.3V via Schottky D22, always on; ~2.85 V at 170 mA on a 3.2 V rail | | | (3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"
Changed lines of the file:
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@@
-		(color 0 0 0 0)
-	)
-	(label "EXT_VP"
-		(at 231.14 58.42 0)
-		(fields_autoplaced yes)
-		(effects
-			(font
-				(size 1.27 1.27)
-			)
-			(justify left bottom)
-		)
-	)
-	(junction
-		(at 242.57 58.42)
-		(diameter 0)
 		(color 0 0 0 0)
 	)
@@
 			(width 0)
 			(type default)
-		)
-	)
-	(label "EXT_VP"
-		(at 193.04 86.36 90)
-		(fields_autoplaced yes)
-		(effects
-			(font
-				(size 1.27 1.27)
-			)
-			(justify left bottom)
 		)
 	)
@@
 		)
 	)
-	(text "External comms port, VE.Direct pinout (plans/ext-comms-port.md)\n\nJ5 pin | signal | dir (Fugu view) | notes\n1 | GND | - | logic GND = Bat-; non-isolated\n2 | RX | in | 3.3 V logic, 5.5 V tolerant (U8), idles high (R50)\n3 | TX | out | 3.3 V push-pull via 220R, Hi-Z unless EXT_TX_OE_N low (R46 pull-up)\n4 | V+ | out | EXT_VP: +3.3V via Schottky D22, always on; ~2.85 V at 170 mA on a 3.2 V rail\n  | | | (3.3 V -3 %, VF ~0.35 V typ); ~2.95 V at a nominal 3.3 V rail\n\nU7 (TX buffer) runs from EXT_VP so TX high = V+: the CAN adapter's ISO1042 has VCC1 = V+ and\nTXD <= VCC1 + 0.5 V. Caveat: a peer that drives pin 4 at 5 V lifts U7 to 5 V, where the 3.3 V /OE\npull-up is below VIH, so TX-off is not guaranteed in that case (plan qualification item 3).\n\nMCU: EXT_TX GPIO36, EXT_RX GPIO37, EXT_TX_OE_N GPIO48\n(not GPIO38/39: driven low in USB-OTG download boot mode, Espressif schematic checklist)\nWrong-adapter protection is in software only (Fab, 2026-09-28/29): no V+ switch, no V+ current sense.\nNo short protection on pin 4 (Fab, 2026-09-29): a short browns out the shared 0.5 A LM5163 rail.\nA PTC cannot help: any PTC holding 0.17 A at 60 C trips at 0.75 A, above the rail's 0.5 A.\nD22 blocks a peer that drives pin 4.\nAdapters draw far more than a Victron port's 10 mA; label them 'Fugu only'."
+	(text "External comms port, VE.Direct pinout (plans/ext-comms-port.md)\n\nJ5 pin | signal | dir (Fugu view) | notes\n1 | GND | - | logic GND = Bat-; non-isolated\n2 | RX | in | 3.3 V logic, 5.5 V tolerant (U8), idles high (R50)\n3 | TX | out | 3.3 V push-pull via 220R, Hi-Z unless EXT_TX_OE_N low (R46 pull-up)\n4 | V+ | out | +3.3V rail direct, always on (Fab, 2026-09-30). C33 at pin 4 = ESD sink + U7 bypass\n\nMCU: EXT_TX GPIO36, EXT_RX GPIO37, EXT_TX_OE_N GPIO48\n(not GPIO38/39: driven low in USB-OTG download boot mode, Espressif schematic checklist)\nWrong-adapter protection is in software only (Fab, 2026-09-28/29): no V+ switch, no V+ current sense.\nNo short protection and no back-feed block on pin 4 (Fab, 2026-09-29/30): a short browns out the\nshared 0.5 A LM5163 rail; a peer driving pin 4 drives the 3.3 V rail.\nAdapters: non-isolated, bus pins rated +/-70 V class (60 V battery GND fault); label them 'Fugu only'."
 		(exclude_from_sim no)
 		(at 20.32 30.48 0)
@@
 	)
 	(symbol
-		(lib_id "Device:D_Schottky")
-		(at 198.12 58.42 180)
-		(unit 1)
-		(body_style 1)
-		(exclude_from_sim no)
-		(in_bom yes)
-		(on_board yes)
-		(in_pos_files yes)
-		(dnp no)
-		(property "Reference" "D22"
-			(at 194.31 53.34 0)
-			(show_name no)
-			(do_not_autoplace no)
-			(effects
-				(font
-					(size 1.27 1.27)
-				)
-				(justify right)
-			)
-		)
-		(property "Value" "MSS1P4-M3/89A"
-			(at 194.31 55.88 0)
-			(show_name no)
-			(do_not_autoplace no)
-			(effects
-				(font
-					(size 1.27 1.27)
-				)
-				(justify right)
-			)
-		)
-		(property "Footprint" "Diode_SMD:D_MicroSMP_LargeCathode"
-			(at 198.12 58.42 0)
-			(hide yes)
-			(show_name no)
-			(do_not_autoplace no)
-			(effects
-				(font
-					(size 1.27 1.27)
-				)
-			)
-		)
-		(property "Datasheet" "https://www.vishay.com/docs/89019/mss1p4.pdf"
-			(at 198.12 58.42 0)
-			(hide yes)
-			(show_name no)
-			(do_not_autoplace no)
-			(effects
-				(font
-					(size 1.27 1.27)
-				)
-			)
-		)
-		(property "Description" ""
-			(at 198.12 58.42 0)
-			(hide yes)
-			(show_name no)
-			(do_not_autoplace no)
-			(effects
-				(font
-					(size 1.27 1.27)
-				)
-			)
-		)
-		(property "MPN" "MSS1P4-M3/89A"
-			(at 198.12 58.42 0)
-			(hide yes)
-			(show_name no)
-			(do_not_autoplace no)
-			(effects
-				(font
-					(size 1.27 1.27)
-				)
-			)
-		)
-		(property "Desc" "ExtPort V+ back-feed block"
-			(at 198.12 58.42 0)
-			(hide yes)
-			(show_name no)
-			(do_not_autoplace no)
-			(effects
-				(font
-					(size 1.27 1.27)
-				)
-			)
-		)
-		(property "Manufacturer" "Vishay"
-			(at 198.12 58.42 0)
-			(hide yes)
-			(show_name no)
-			(do_not_autoplace no)
-			(effects
-				(font
-					(size 1.27 1.27)
-				)
-			)
-		)
-		(pin "1"
-		)
-		(pin "2"
-		)
-		(instances
-			(project "Fugu2"
-				(path "/e6692049-eaa1-423b-b1ac-05fb6d0f1fc2/cb058d3e-80b8-7be1-708b-f93a7279feab"
-					(reference "D22")
-					(unit 1)
-				)
-			)
-		)
-	)
-	(symbol
 		(lib_id "Device:C_Small")
 		(at 218.44 63.5 0)
@@
 	)
 	(symbol
-		(lib_id "power:PWR_FLAG")
-		(at 242.57 58.42 0)
-		(unit 1)
-		(body_style 1)
-		(exclude_from_sim no)
-		(in_bom yes)
-		(on_board yes)
-		(in_pos_files yes)
-		(dnp no)
-		(property "Reference" "#FLG101"
-			(at 242.57 62.23 0)
-			(hide yes)
-			(show_name no)
-			(do_not_autoplace no)
-			(effects
-				(font
-					(size 1.27 1.27)
-				)
-			)
-		)
-		(property "Value" "PWR_FLAG"
-			(at 242.57 54.61 0)
-			(show_name no)
-			(do_not_autoplace no)
-			(effects
-				(font
-					(size 1.27 1.27)
-				)
-			)
-		)
-		(property "Footprint" ""
-			(at 242.57 58.42 0)
-			(hide yes)
-			(show_name no)
-			(do_not_autoplace no)
-			(effects
-				(font
-					(size 1.27 1.27)
-				)
-			)
-		)
-		(property "Datasheet" ""
-			(at 242.57 58.42 0)
-			(hide yes)
-			(show_name no)
-			(do_not_autoplace no)
-			(effects
-				(font
-					(size 1.27 1.27)
-				)
-			)
-		)
-		(property "Description" ""
-			(at 242.57 58.42 0)
-			(hide yes)
-			(show_name no)
-			(do_not_autoplace no)
-			(effects
-				(font
-					(size 1.27 1.27)
-				)
-			)
-		)
-		(pin "1"
-		)
-		(instances
-			(project "Fugu2"
-				(path "/e6692049-eaa1-423b-b1ac-05fb6d0f1fc2/cb058d3e-80b8-7be1-708b-f93a7279feab"
-					(reference "#FLG101")
-					(unit 1)
-				)
-			)
-		)
-	)
-	(symbol
 		(lib_id "74xGxx:74LVC1G125")
 		(at 198.12 99.06 0)
@@
 					(unit 1)
 				)
+			)
+		)
+	)
+	(wire
+		(pts
+			(xy 194.31 58.42) (xy 201.93 58.42)
+		)
+		(stroke
+			(width 0)
+			(type default)
+		)
+	)
+	(symbol
+		(lib_id "power:+3.3V")
+		(at 193.04 86.36 0)
+		(unit 1)
+		(body_style 1)
+		(exclude_from_sim no)
+		(in_bom yes)
+		(on_board yes)
+		(in_pos_files yes)
+		(dnp no)
+		(property "Reference" "#PWR113"
+			(at 193.04 90.17 0)
+			(hide yes)
+			(show_name no)
+			(do_not_autoplace no)
+			(effects
+				(font
+					(size 1.27 1.27)
+				)
+			)
+		)
+		(property "Value" "+3.3V"
+			(at 193.04 82.55 0)
+			(show_name no)
+			(do_not_autoplace no)
+			(effects
+				(font
+					(size 1.27 1.27)
+				)
+			)
+		)
+		(property "Footprint" ""
+			(at 193.04 86.36 0)
+			(hide yes)
+			(show_name no)
+			(do_not_autoplace no)
+			(effects
+				(font
+					(size 1.27 1.27)
+				)
+			)
+		)
+		(property "Datasheet" ""
+			(at 193.04 86.36 0)
+			(hide yes)
+			(show_name no)
+			(do_not_autoplace no)
+			(effects
+				(font
+					(size 1.27 1.27)
+				)
+			)
+		)
+		(property "Description" ""
+			(at 193.04 86.36 0)
+			(hide yes)
+			(show_name no)
+			(do_not_autoplace no)
+			(effects
+				(font
+					(size 1.27 1.27)
+				)
+			)
+		)
+		(pin "1"
+		)
+		(instances
+			(project "Fugu2"
+				(path "/e6692049-eaa1-423b-b1ac-05fb6d0f1fc2/cb058d3e-80b8-7be1-708b-f93a7279feab"
+					(reference "#PWR113")
+					(unit 1)
+				)
