File: PowerStage.kicad_sch (KiCad schematic)
At the start: 48 parts, among them J10 691256610002, J3 Conn_L_SW, J6 Conn_L_out, J9 691256610002, Q1 IPA050N10NM5S, Q10 IPP022N12NM6, Q2 IPP022N12NM6, Q3 IPA050N10NM5S, Q5 TPH1R306PL,L1Q or NTMFS5C612N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, Q6 TPH1R306PL,L1Q or NTMFS5C612N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, Q7 TPH1R306PL,L1Q or NTMFS5C612N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

Commit message: Cin: 3x Chemi-Con KZN 1000uF (C11, C12, new C34); C10 is Cout, also KZN
Only caps on Solar+ are Cin. C10 sits on BflowS (inductor output) and is
Cout, so the old board had just two input electrolytics, each carrying
~8 A rms at 33 A (~3.5x a ZLH 470uF rating).

- C11, C12, C34 (Solar+) and C10 (BflowS): 1000uF 100V, 18 mm / 7.5 mm
  footprint (C11 was 16 mm), Chemi-Con EKZN101ELL102MM40S (DigiKey
  565-4153-ND) recorded in Description, Manufacturer and Digikey. MPN stays
  DNP (hand-assembled; PCBWay reads DNP as "do not mount").
- C10 Desc: Cin -> Cout.
- doc/Capacitors.md: new "Input bulk decision (2026-10-04)" section with
  ripple math (16.06 A), part choice, rejected options (UBY, TDK B41793,
  snap-ins, hybrids), Chemi-Con lower-ambient guidance, open items
  (KZN dT limit, layout spacing), the Outback FM40 comparison, and a fix to
  the ZLJ 680uF 18x35.5 row (3.51 A / 27 mOhm).

Reviewed by two independent Codex runs (~/codex-reviews/fugu2-cin-caps*).
The PCB still needs updating from the schematic: C11 footprint, add C34,
resolve the orphan C12 footprint, and space the 18 mm cans >= ~19 mm apart.
Parts:
- added C34: 1000uF, 100V, Capacitor_THT:CP_Radial_D18.0mm_P7.50mm, symbol Device:C_Polarized
- C10: value 470uF, 100V -> 1000uF, 100V; Desc Cin -> Cout; Digikey (none) -> 565-4153-ND; Manufacturer (none) -> Chemi-Con
- C11: value 470uF, 100V -> 1000uF, 100V; footprint Capacitor_THT:CP_Radial_D16.0mm_P7.50mm -> Capacitor_THT:CP_Radial_D18.0mm_P7.50mm; Digikey (none) -> 565-4153-ND; Manufacturer (none) -> Chemi-Con
- C12: value 470uF, 100V -> 1000uF, 100V; Digikey (none) -> 565-4153-ND; Manufacturer (none) -> Chemi-Con
Connections:
- net BuckGND: now also C34.2
- net Solar+: now also C34.1
Changed lines of the file:
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@@
 	)
 	(junction
+		(at 48.895 77.47)
+		(diameter 0)
+		(color 0 0 0 0)
+	)
+	(junction
 		(at 135.255 51.435)
 		(diameter 0)
@@
 	)
 	(junction
+		(at 48.895 34.29)
+		(diameter 0)
+		(color 0 0 0 0)
+	)
+	(junction
 		(at 70.485 114.935)
 		(diameter 0)
@@
 	(wire
 		(pts
+			(xy 48.895 34.29) (xy 48.895 38.735)
+		)
+		(stroke
+			(width 0)
+			(type default)
+		)
+	)
+	(wire
+		(pts
 			(xy 48.895 98.425) (xy 59.055 98.425)
 		)
@@
 	(wire
 		(pts
+			(xy 48.895 34.29) (xy 54.61 34.29)
+		)
+		(stroke
+			(width 0)
+			(type default)
+		)
+	)
+	(wire
+		(pts
 			(xy 86.36 51.435) (xy 91.44 51.435)
 		)
@@
 	(wire
 		(pts
-			(xy 44.45 34.29) (xy 54.61 34.29)
+			(xy 44.45 34.29) (xy 48.895 34.29)
 		)
 		(stroke
@@
 	(wire
 		(pts
+			(xy 48.895 46.355) (xy 48.895 77.47)
+		)
+		(stroke
+			(width 0)
+			(type default)
+		)
+	)
+	(wire
+		(pts
 			(xy 75.565 41.91) (xy 75.565 46.99)
 		)
@@
 	(wire
 		(pts
-			(xy 44.45 77.47) (xy 54.61 77.47)
+			(xy 44.45 77.47) (xy 48.895 77.47)
 		)
 		(stroke
@@
 	(wire
 		(pts
+			(xy 48.895 77.47) (xy 54.61 77.47)
+		)
+		(stroke
+			(width 0)
+			(type default)
+		)
+	)
+	(wire
+		(pts
 			(xy 57.15 59.69) (xy 54.61 59.69)
 		)
@@
 			)
 		)
-		(property "Value" "470uF, 100V"
+		(property "Value" "1000uF, 100V"
 			(at 43.18 67.31 90)
 			(show_name no)
@@
 			)
 		)
-		(property "Datasheet" ""
+		(property "Datasheet" "https://www.chemi-con.co.jp/products/relatedfiles/capacitor/catalog/KZNLL-e.PDF"
 			(at 44.45 53.34 0)
 			(hide yes)
@@
 			)
 		)
-		(property "Description" ""
+		(property "Description" "Chemi-Con EKZN101ELL102MM40S (hand-assembled, MPN=DNP for fab BOM)"
 			(at 44.45 53.34 0)
 			(hide yes)
@@
 			)
 		)
-		(property "Manufacturer" ""
+		(property "Manufacturer" "Chemi-Con"
 			(at 44.45 53.34 0)
 			(hide yes)
@@
 			)
 		)
-		(property "Digikey" ""
+		(property "Digikey" "565-4153-ND"
 			(at 44.45 53.34 0)
 			(hide yes)
@@
 			)
 		)
-		(property "Value" "470uF, 100V"
+		(property "Value" "1000uF, 100V"
 			(at 35.56 67.945 90)
 			(show_name no)
@@
 			)
 		)
-		(property "Footprint" "Capacitor_THT:CP_Radial_D16.0mm_P7.50mm"
+		(property "Footprint" "Capacitor_THT:CP_Radial_D18.0mm_P7.50mm"
 			(at 37.7952 57.15 0)
 			(hide yes)
@@
 			)
 		)
-		(property "Datasheet" ""
+		(property "Datasheet" "https://www.chemi-con.co.jp/products/relatedfiles/capacitor/catalog/KZNLL-e.PDF"
 			(at 36.83 53.34 0)
 			(hide yes)
@@
 			)
 		)
-		(property "Description" ""
+		(property "Description" "Chemi-Con EKZN101ELL102MM40S (hand-assembled, MPN=DNP for fab BOM)"
 			(at 36.83 53.34 0)
 			(hide yes)
@@
 			)
 		)
-		(property "Manufacturer" ""
+		(property "Manufacturer" "Chemi-Con"
 			(at 36.83 53.34 0)
 			(hide yes)
@@
 			)
 		)
-		(property "Digikey" ""
+		(property "Digikey" "565-4153-ND"
 			(at 36.83 53.34 0)
 			(hide yes)
@@
 			)
 		)
-		(property "Value" "470uF, 100V"
+		(property "Value" "1000uF, 100V"
 			(at 130.175 64.135 0)
 			(show_name no)
@@
 			)
 		)
-		(property "Datasheet" ""
+		(property "Datasheet" "https://www.chemi-con.co.jp/products/relatedfiles/capacitor/catalog/KZNLL-e.PDF"
 			(at 130.175 61.595 0)
 			(hide yes)
@@
 			)
 		)
-		(property "Description" ""
+		(property "Description" "Chemi-Con EKZN101ELL102MM40S (hand-assembled, MPN=DNP for fab BOM)"
 			(at 130.175 61.595 0)
 			(hide yes)
@@
 			)
 		)
-		(property "Desc" "Cin"
+		(property "Desc" "Cout"
 			(at 130.175 61.595 0)
 			(hide yes)
@@
 			)
 		)
-		(property "Manufacturer" ""
+		(property "Manufacturer" "Chemi-Con"
 			(at 130.175 61.595 0)
 			(hide yes)
@@
 			)
 		)
-		(property "Digikey" ""
+		(property "Digikey" "565-4153-ND"
 			(at 130.175 61.595 0)
 			(hide yes)
@@
 					(unit 1)
 				)
+			)
+		)
+	)
+	(symbol
+		(lib_id "Device:C_Polarized")
+		(at 48.895 42.545 0)
+		(unit 1)
+		(body_style 1)
+		(exclude_from_sim no)
+		(in_bom yes)
+		(on_board yes)
+		(in_pos_files yes)
+		(dnp no)
+		(property "Reference" "C34"
+			(at 48.895 40.005 0)
+			(show_name no)
+			(do_not_autoplace no)
+			(effects
+				(font
+					(size 1.27 1.27)
+				)
+				(justify left)
+			)
+		)
+		(property "Value" "1000uF, 100V"
+			(at 47.625 56.515 90)
+			(show_name no)
+			(do_not_autoplace no)
+			(effects
+				(font
+					(size 1.27 1.27)
+				)
+				(justify left)
+			)
+		)
+		(property "Footprint" "Capacitor_THT:CP_Radial_D18.0mm_P7.50mm"
+			(at 49.8602 46.355 0)
+			(hide yes)
+			(show_name no)
+			(do_not_autoplace no)
+			(effects
+				(font
+					(size 1.27 1.27)
+				)
+			)
+		)
+		(property "Datasheet" "https://www.chemi-con.co.jp/products/relatedfiles/capacitor/catalog/KZNLL-e.PDF"
+			(at 48.895 42.545 0)
+			(hide yes)
+			(show_name no)
+			(do_not_autoplace no)
+			(effects
+				(font
+					(size 1.27 1.27)
+				)
+			)
+		)
+		(property "Description" "Chemi-Con EKZN101ELL102MM40S (hand-assembled, MPN=DNP for fab BOM)"
+			(at 48.895 42.545 0)
+			(hide yes)
+			(show_name no)
+			(do_not_autoplace no)
+			(effects
+				(font
+					(size 1.27 1.27)
+				)
+			)
+		)
+		(property "MPN" "DNP"
+			(at 48.895 42.545 0)
+			(hide yes)
+			(show_name no)
+			(do_not_autoplace no)
+			(effects
+				(font
+					(size 1.27 1.27)
+				)
+			)
+		)
+		(property "Desc" "Cin"
+			(at 48.895 42.545 0)
+			(hide yes)
+			(show_name no)
+			(do_not_autoplace no)
+			(effects
+				(font
+					(size 1.27 1.27)
+				)
+			)
+		)
+		(property "Manufacturer" "Chemi-Con"
+			(at 48.895 42.545 0)
+			(hide yes)
+			(show_name no)
+			(do_not_autoplace no)
+			(effects
+				(font
+					(size 1.27 1.27)
+				)
+			)
+		)
+		(property "Digikey" "565-4153-ND"
+			(at 48.895 42.545 0)
+			(hide yes)
+			(show_name no)
+			(do_not_autoplace no)
+			(effects
+				(font
+					(size 1.27 1.27)
+				)
+			)
+		)
+		(pin "1"
+		)
+		(pin "2"
+		)
+		(instances
+			(project "Fugu2"
+				(path "/e6692049-eaa1-423b-b1ac-05fb6d0f1fc2/13b9cc5d-522a-5e4c-97c3-f9530ebe4903"
+					(reference "C34")
+					(unit 1)
+				)
